File: dnafh/board/definitely_not_a_fire_hazard.sch (KiCad schematic (older format))
At the start: 32 parts, among them IC1 ATTINY85-S, P1 USB_OTG_B, P2 CONN_01X01_WS2812, P3 PB1, P4 CONN_BAT+, P5 CONN_BAT-, P6 CONN_LEDVCC, P7 PB2, Q1 ML8205A, Q2 IRLML6401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

Commit message: board changes and fixes
Parts:
- P1: symbol USB_OTG -> USB_OTG-RESCUE-definitely_not_a_fire_hazard
- R3: value 220 -> 100
- R4: value 100 -> 500
- SW1: symbol SW_SPST -> SW_SPST-RESCUE-definitely_not_a_fire_hazard
Other:
- note added: "TODO:\n* CE von 4056 an pulldown"
Changed lines of the file:
@@
 P 3550 1400
 F 0 "R3" V 3600 1550 50  0000 C CNN
-F 1 "220" V 3550 1400 50  0000 C CNN
+F 1 "100" V 3550 1400 50  0000 C CNN
 F 2 "Resistors_SMD:R_0805" V 3480 1400 50  0001 C CNN
 F 3 "" H 3550 1400 50  0000 C CNN
@@
 P 3550 1600
 F 0 "R4" V 3600 1750 50  0000 C CNN
-F 1 "100" V 3550 1600 50  0000 C CNN
+F 1 "500" V 3550 1600 50  0000 C CNN
 F 2 "Resistors_SMD:R_0805" V 3480 1600 50  0001 C CNN
 F 3 "" H 3550 1600 50  0000 C CNN
@@
 Li-Ion Charger
 $Comp
-L USB_OTG P1
+L USB_OTG-RESCUE-definitely_not_a_fire_hazard P1
 U 1 1 58963CCF
 P 800 1700
@@
 Connection ~ 4000 3050
 Wire Wire Line
-	4750 2650 4450 2650
-Connection ~ 4450 2650
-Wire Wire Line
 	5100 2300 5100 3050
 Wire Notes Line
@@
 Connection ~ 5100 2350
 Wire Wire Line
-	5100 2000 5100 1900
-Wire Wire Line
-	5100 1900 4450 1900
+	5100 1900 5100 2000
+Wire Wire Line
+	4450 1900 5100 1900
 Connection ~ 4450 1900
 Connection ~ 4450 1500
@@
 	4950 1250 5150 1250
 $Comp
-L SW_SPST SW1
+L SW_SPST-RESCUE-definitely_not_a_fire_hazard SW1
 U 1 1 58A755AE
 P 6700 4850
@@
 	-1   0    0    1
 $EndComp
+Wire Wire Line
+	4750 2650 4450 2650
+Connection ~ 4450 2650
+Text Notes 5750 1350 0    60   ~ 0
+TODO:\n* CE von 4056 an pulldown
 $EndSCHEMATC
